Commit message: The mini is smaller

File: mini_control/description/urdf/rrbot_macro.urdf.xacro (robot description, xacro)
@@ -10,28 +10,25 @@
   <link name="${prefix}base_link">
     <collision>
-      <origin xyz="0 0 1" rpy="0 0 0"/>
+      <origin xyz="0.0 0.0 0.25" rpy="0 0 0"/>
       <geometry>
-        <box size="0.1 0.1 2"/>
+        <box size="0.025 0.025 0.5"/>
       </geometry>
     </collision>
     <visual>
-      <origin xyz="0 0 1" rpy="0 0 0"/>
+      <origin xyz="0.0 0.0 0.25" rpy="0 0 0"/>
       <geometry>
-        <box size="0.1 0.1 2"/>
+        <box size="0.025 0.025 0.5"/>
       </geometry>
     </visual>
-    <inertial>
-      <origin xyz="0 0 1" rpy="0 0 0"/>
-      <mass value="2"/>
-      <inertia
-        ixx="0.01" ixy="0.0" ixz="0.0"
-        iyy="0.01" iyz="0.0"
-        izz="0.01"/>
-    </inertial>
+      <inertial>
+        <origin xyz="0.0 0.0 0.0" rpy="0 0 0"/>
+        <mass value="0.5"/>
+        <inertia ixx="0.001" ixy="0.0" ixz="0.0" iyy="0.001" iyz="0.0" izz="0.001"/>
+      </inertial>
   </link>
   <joint name="${prefix}joint1" type="revolute">
     <parent link="${prefix}base_link"/>
     <child link="${prefix}link1"/>
-    <origin xyz="0 0.1 1.95" rpy="0 0 0"/>
+    <origin xyz="0.0 0.025 0.4875" rpy="0 0 0"/>
     <axis xyz="0 1 0"/>
     <dynamics damping="0.8"/>
@@ -41,28 +38,25 @@
   <link name="${prefix}link1">
     <collision>
-      <origin xyz="0 0 0.45" rpy="0 0 0"/>
+      <origin xyz="0.0 0.0 0.1125" rpy="0 0 0"/>
       <geometry>
-        <box size="0.1 0.1 1"/>
+        <box size="0.025 0.025 0.25"/>
       </geometry>
     </collision>
     <visual>
-      <origin xyz="0 0 0.45" rpy="0 0 0"/>
+      <origin xyz="0.0 0.0 0.1125" rpy="0 0 0"/>
       <geometry>
-        <box size="0.1 0.1 1"/>
+        <box size="0.025 0.025 0.25"/>
       </geometry>
     </visual>
-    <inertial>
-      <origin xyz="0 0 0.45" rpy="0 0 0"/>
-      <mass value="1"/>
-      <inertia
-        ixx="0.01" ixy="0.0" ixz="0.0"
-        iyy="0.01" iyz="0.0"
-        izz="0.01"/>
-    </inertial>
+      <inertial>
+        <origin xyz="0.0 0.0 0.0" rpy="0 0 0"/>
+        <mass value="0.5"/>
+        <inertia ixx="0.001" ixy="0.0" ixz="0.0" iyy="0.001" iyz="0.0" izz="0.001"/>
+      </inertial>
   </link>
   <joint name="${prefix}joint2" type="revolute">
     <parent link="${prefix}link1"/>
     <child link="${prefix}link2"/>
-    <origin xyz="0 0.1 0.95" rpy="0 0 0"/>
+    <origin xyz="0.0 0.025 0.2375" rpy="0 0 0"/>
     <axis xyz="0 1 0"/>
     <dynamics damping="0.8"/>
@@ -72,23 +66,20 @@
   <link name="${prefix}link2">
     <collision>
-      <origin xyz="0 0 0.45" rpy="0 0 0"/>
+      <origin xyz="0.0 0.0 0.1125" rpy="0 0 0"/>
       <geometry>
-        <box size="0.1 0.1 1"/>
+        <box size="0.025 0.025 0.25"/>
       </geometry>
     </collision>
     <visual>
-      <origin xyz="0 0 0.45" rpy="0 0 0"/>
+      <origin xyz="0.0 0.0 0.1125" rpy="0 0 0"/>
       <geometry>
-        <box size="0.1 0.1 1"/>
+        <box size="0.025 0.025 0.25"/>
       </geometry>
     </visual>
-    <inertial>
-      <origin xyz="0 0 0.45" rpy="0 0 0"/>
-      <mass value="1"/>
-      <inertia
-        ixx="0.01" ixy="0.0" ixz="0.0"
-        iyy="0.01" iyz="0.0"
-        izz="0.01"/>
-    </inertial>
+      <inertial>
+        <origin xyz="0.0 0.0 0.0" rpy="0 0 0"/>
+        <mass value="0.5"/>
+        <inertia ixx="0.001" ixy="0.0" ixz="0.0" iyy="0.001" iyz="0.0" izz="0.001"/>
+      </inertial>
   </link>
   </xacro:macro>

Commit message: Just corrected the inertia

File: mini_control/description/urdf/rrbot_macro.urdf.xacro (robot description, xacro)
@@ -24,5 +24,7 @@
         <origin xyz="0.0 0.0 0.0" rpy="0 0 0"/>
         <mass value="0.5"/>
-        <inertia ixx="0.001" ixy="0.0" ixz="0.0" iyy="0.001" iyz="0.0" izz="0.001"/>
+        <inertia
+          ixx="0.010443" ixy="0.0" ixz="0.0"
+          iyy="0.010443" iyz="0.0" izz="0.0000521"/>
       </inertial>
   </link>
@@ -52,5 +54,7 @@
         <origin xyz="0.0 0.0 0.0" rpy="0 0 0"/>
         <mass value="0.5"/>
-        <inertia ixx="0.001" ixy="0.0" ixz="0.0" iyy="0.001" iyz="0.0" izz="0.001"/>
+        <inertia
+          ixx="0.00263" ixy="0.0" ixz="0.0"
+          iyy="0.00263" iyz="0.0" izz="0.0000521"/>
       </inertial>
   </link>
@@ -80,5 +84,7 @@
         <origin xyz="0.0 0.0 0.0" rpy="0 0 0"/>
         <mass value="0.5"/>
-        <inertia ixx="0.001" ixy="0.0" ixz="0.0" iyy="0.001" iyz="0.0" izz="0.001"/>
+        <inertia
+          ixx="0.00263" ixy="0.0" ixz="0.0"
+          iyy="0.00263" iyz="0.0" izz="0.0000521"/>
       </inertial>
   </link>
