Commit message: Added new rrbot.urdf .

File: mini_control/description/urdf/rrbot.urdf.xacro (robot description, xacro)
@@ -1,5 +1,5 @@
 <?xml version="1.0"?>
 <robot xmlns:xacro="http://www.ros.org/wiki/xacro" name="rrbot">
-  <xacro:include filename="$(find mini_control)/description/urdf/rrbot_macro.urdf.xacro" />
+  <xacro:include filename="$(find mini_control)/description/urdf/rrbot_macro_2.urdf.xacro" />
   <!--Here I changed "world" to iiwa_tool0, the last link from my KUKA-->
   <!--link name="world"-->

File: mini_control/description/urdf/rrbot_.urdf (robot description, URDF)
Before this commit: robot rrbot2, 4 links, 3 joints
Links:
- removed link world
- added link tool0
Joints:
- joint base_joint: parent world -> tool0

File: mini_control/description/urdf/rrbot_macro_2.urdf.xacro (robot description, xacro)
@@ -10,5 +10,5 @@
   <link name="${prefix}base_link">
     <collision>
-      <origin xyz="0 0 0.025" rpy="0 0 0"/>
+      <origin xyz="0 0 0.25" rpy="0 0 0"/>
       <geometry>
         <box size="0.025 0.025 0.5"/>
@@ -16,5 +16,5 @@
     </collision>
     <visual>
-      <origin xyz="0 0 0.025" rpy="0 0 0"/>
+      <origin xyz="0 0 0.25" rpy="0 0 0"/>
       <geometry>
         <box size="0.025 0.025 0.5"/>
@@ -22,5 +22,5 @@
     </visual>
     <inertial>
-      <origin xyz="0 0 0.025" rpy="0 0 0"/>
+      <origin xyz="0 0 0.25" rpy="0 0 0"/>
       <mass value="0.5"/>
       <inertia
@@ -33,5 +33,5 @@
     <parent link="${prefix}base_link"/>
     <child link="${prefix}link1"/>
-    <origin xyz="0 0.025 0.45" rpy="0 0 0"/>
+    <origin xyz="0 0.025 0.48" rpy="0 0 0"/>
     <axis xyz="0 1 0"/>
     <dynamics damping="0.8"/>
@@ -41,5 +41,5 @@
   <link name="${prefix}link1">
     <collision>
-      <origin xyz="0 0 0.2" rpy="0 0 0"/>
+      <origin xyz="0 0 0.1" rpy="0 0 0"/>
       <geometry>
         <box size="0.025 0.025 0.25"/>
@@ -47,5 +47,5 @@
     </collision>
     <visual>
-      <origin xyz="0 0 0.2" rpy="0 0 0"/>
+      <origin xyz="0 0 0.1" rpy="0 0 0"/>
       <geometry>
         <box size="0.025 0.025 0.25"/>
@@ -53,5 +53,5 @@
     </visual>
     <inertial>
-      <origin xyz="0 0 0.2" rpy="0 0 0"/>
+      <origin xyz="0 0 0.1" rpy="0 0 0"/>
       <mass value="0.25"/>
       <inertia
@@ -64,5 +64,5 @@
     <parent link="${prefix}link1"/>
     <child link="${prefix}link2"/>
-    <origin xyz="0 0.025 0.075" rpy="0 0 0"/>
+    <origin xyz="0 0.025 0.2" rpy="0 0 0"/>
     <axis xyz="0 1 0"/>
     <dynamics damping="0.8"/>
@@ -72,5 +72,5 @@
   <link name="${prefix}link2">
     <collision>
-      <origin xyz="0 0 0.2" rpy="0 0 0"/>
+      <origin xyz="0 0 0.1" rpy="0 0 0"/>
       <geometry>
         <box size="0.025 0.025 0.25"/>
@@ -78,5 +78,5 @@
     </collision>
     <visual>
-      <origin xyz="0 0 0.2" rpy="0 0 0"/>
+      <origin xyz="0 0 0.1" rpy="0 0 0"/>
       <geometry>
         <box size="0.025 0.025 0.25"/>
@@ -84,6 +84,6 @@
     </visual>
     <inertial>
-      <origin xyz="0 0 0.2" rpy="0 0 0"/>
-      <mass value="0.25"/>
+      <origin xyz="0 0 0.1" rpy="0 0 0"/>
+      <mass value="1"/>
       <inertia
         ixx="0.01" ixy="0.0" ixz="0.0"
